Commit message: change path of mesh file to original

File: ur5_data_collect_fw/urdf/3finger.urdf (robot description, URDF)
Before this commit: robot None, 24 links, 24 joints
Links:
- link H1_F1_base_link: geometry collision mesh filename=package://fh_desc/meshes/v2/finger_base_link_simple.dae; visual mesh filename=package://fh_desc/meshes/v2/finger_base_link_simple.dae
- link H1_F1_link_1: geometry collision mesh filename=package://fh_desc/meshes/v2/finger_prox_link_simple.dae; visual mesh filename=package://fh_desc/meshes/v2/finger_prox_link_simple.dae
- link H1_F1_link_2: geometry collision mesh filename=package://fh_desc/meshes/v2/finger_dist_link_simple.dae; visual mesh filename=package://fh_desc/meshes/v2/finger_dist_link_simple.dae
- link H1_F1_palm_link: geometry visual mesh filename=package://fh_desc/meshes/v2/finger_palm_link.dae
- link H1_F1_tip: geometry collision mesh filename=package://fh_desc/meshes/omd-d18-tip.dae; visual mesh filename=package://fh_desc/meshes/omd-d18-tip.dae
- link H1_F2_base_link: geometry collision mesh filename=package://fh_desc/meshes/v2/finger_base_link_simple.dae; visual mesh filename=package://fh_desc/meshes/v2/finger_base_link_simple.dae
- link H1_F2_link_1: geometry collision mesh filename=package://fh_desc/meshes/v2/finger_prox_link_simple.dae; visual mesh filename=package://fh_desc/meshes/v2/finger_prox_link_simple.dae
- link H1_F2_link_2: geometry collision mesh filename=package://fh_desc/meshes/v2/finger_dist_link_simple.dae; visual mesh filename=package://fh_desc/meshes/v2/finger_dist_link_simple.dae
- link H1_F2_palm_link: geometry visual mesh filename=package://fh_desc/meshes/v2/finger_palm_link.dae
- link H1_F2_tip: geometry collision mesh filename=package://fh_desc/meshes/omd-d18-tip.dae; visual mesh filename=package://fh_desc/meshes/omd-d18-tip.dae
- link H1_F3_base_link: geometry collision mesh filename=package://fh_desc/meshes/v2/finger_base_link_simple.dae; visual mesh filename=package://fh_desc/meshes/v2/finger_base_link_simple.dae
- link H1_F3_link_1: geometry collision mesh filename=package://fh_desc/meshes/v2/finger_prox_link_simple.dae; visual mesh filename=package://fh_desc/meshes/v2/finger_prox_link_simple.dae
- link H1_F3_link_2: geometry collision mesh filename=package://fh_desc/meshes/v2/finger_dist_link_simple.dae; visual mesh filename=package://fh_desc/meshes/v2/finger_dist_link_simple.dae
- link H1_F3_palm_link: geometry visual mesh filename=package://fh_desc/meshes/v2/finger_palm_link.dae
- link H1_F3_tip: geometry collision mesh filename=package://fh_desc/meshes/omd-d18-tip.dae; visual mesh filename=package://fh_desc/meshes/omd-d18-tip.dae
- link H1_base_link: geometry collision mesh filename=package://fh_desc/meshes/v2/palm_link_simple.dae; visual mesh filename=package://fh_desc/meshes/v2/palm_link_simple.dae
